Commit message: sleep fix

File: urdf/piper_description.urdf (robot description, URDF)
Before this commit: robot piper, 11 links, 10 joints
Links:
- link base_link: geometry collision mesh filename=link0.stl; visual mesh filename=link0.stl
- link gripper_base: geometry collision mesh filename=gripper_base.stl; visual mesh filename=gripper_base.stl
- link link1: geometry collision mesh filename=link1.stl; visual mesh filename=link1.stl
- link link2: geometry collision mesh filename=link2.stl; visual mesh filename=link2.stl
- link link3: geometry collision mesh filename=link3.stl; visual mesh filename=link3.stl
- link link4: geometry collision mesh filename=link4.stl; visual mesh filename=link4.stl
- link link5: geometry collision mesh filename=link5.stl; visual mesh filename=link5.stl
- link link6: geometry collision mesh filename=link6.stl; visual mesh filename=link6.stl
- link link7: geometry collision mesh filename=link7.stl; visual mesh filename=link7.stl
- link link8: geometry collision mesh filename=link8.stl; visual mesh filename=link8.stl
