Commit message: add gripper to cone-e urdfs

File: urdf/piper_cone-e_left.urdf (robot description, URDF)
Before this commit: robot piper, 8 links, 7 joints
Links:
- added link gripper_base, mass 0.18; collision mesh filename=package://piper_description/meshes/gripper_base.STL; visual mesh filename=package://piper_description/meshes/gripper_base.STL
- added link link7, mass 0.025; collision mesh filename=package://piper_description/meshes/link7.STL; visual mesh filename=package://piper_description/meshes/link7.STL
- added link link8, mass 0.025; collision mesh filename=package://piper_description/meshes/link8.STL; visual mesh filename=package://piper_description/meshes/link8.STL
Joints:
- added joint joint6_to_gripper_base: type fixed, parent link6, child gripper_base, origin xyz=0 0 0 rpy=0 0 0
- added joint joint7: type fixed, parent gripper_base, child link7, origin xyz=0 0 0.1358 rpy=1.5708 0 0, axis 0 0 1, limit lower=0 upper=0.035 effort=10 velocity=1
- added joint joint8: type fixed, parent gripper_base, child link8, origin xyz=0 0 0.1358 rpy=1.5708 0 -3.1416, axis 0 0 -1, limit lower=-0.035 upper=0 effort=10 velocity=1

File: urdf/piper_cone-e_right.urdf (robot description, URDF)
Before this commit: robot piper, 8 links, 7 joints
Links:
- added link gripper_base, mass 0.18; collision mesh filename=package://piper_description/meshes/gripper_base.STL; visual mesh filename=package://piper_description/meshes/gripper_base.STL
- added link link7, mass 0.025; collision mesh filename=package://piper_description/meshes/link7.STL; visual mesh filename=package://piper_description/meshes/link7.STL
- added link link8, mass 0.025; collision mesh filename=package://piper_description/meshes/link8.STL; visual mesh filename=package://piper_description/meshes/link8.STL
Joints:
- added joint joint6_to_gripper_base: type fixed, parent link6, child gripper_base, origin xyz=0 0 0 rpy=0 0 0
- added joint joint7: type fixed, parent gripper_base, child link7, origin xyz=0 0 0.1358 rpy=1.5708 0 0, axis 0 0 1, limit lower=0 upper=0.035 effort=10 velocity=1
- added joint joint8: type fixed, parent gripper_base, child link8, origin xyz=0 0 0.1358 rpy=1.5708 0 -3.1416, axis 0 0 -1, limit lower=-0.035 upper=0 effort=10 velocity=1

Commit message: tuned for grav compy of nyu gripper w/o iphone

File: urdf/piper_cone-e_left.urdf (robot description, URDF)
Before this commit: robot piper, 11 links, 10 joints
Links:
- link gripper_base: mass 0.18 -> 0.25
- link link7: mass 0.025 -> 0.01
- link link8: mass 0.025 -> 0.01
